File: toyota_steering_sensor/kicad/toyota-angle-sensor.kicad_pcb (KiCad board)
At the start: 2 copper layers, 161.8 x 161.8 mm, 32 parts, among them IC1 ATMEGA328P-AU, J1 AVR-ISP-6, J2 RJ45, U1 LM7805_TO220, U2 FTDI, U3 LS7366R, U4 MCP2515-xST, U5 AS5047P, U6 TJA1050, Y1 16MHz, Y2 40MHz, Y3 20MHz

Commit message: done routing v2
Parts:
- C10, C11: moved to F.Cu
- R3: moved to B.Cu
- moved C9 48.6 mm to (-3.60, 4.20), turned to 90 degrees
- moved C12 46.5 mm to (-0.40, -6.81), turned to 270 degrees
- moved C10 41.2 mm to (-9.60, -7.40), turned to 0 degrees
- moved C11 37.6 mm to (-9.60, -5.80), turned to 0 degrees
- moved R3 31.0 mm to (-6.60, -10.0)
- moved D2 22.2 mm to (-7.50, -9.50)
- moved Y3 4.12 mm to (-3.60, -6.00), turned to 90 degrees
- moved R4 0.45 mm to (-9.20, 8.40)
- turned C7 to 90 degrees
Connections:
- D2 pad 1: Net-(D2-Pad1) -> GND
- D2 pad 2: /D13,SCK -> Net-(D2-Pad2)
- R3 pad 1: Net-(D2-Pad1) -> /D13,SCK
- R3 pad 2: GND -> Net-(D2-Pad2)
Routing:
- net +5V: track 77.0 -> 106.0 mm, vias 5 -> 6
- net /D13,SCK: track 29.1 -> 39.4 mm, vias 1 -> 3
- net Net-(R5-Pad2): track 0.00 -> 7.13 mm, vias 0 -> 1
- net Net-(C7-Pad2): track 0.00 -> 5.15 mm
- net Net-(U4-Pad8): track 0.00 -> 4.79 mm
- net Net-(U4-Pad9): track 0.00 -> 4.06 mm
- net GND: track 40.5 -> 37.3 mm, vias 8 -> 21
- net Net-(D2-Pad2): track 0.00 -> 2.13 mm, vias 0 -> 1
- net Net-(U4-Pad2): track 3.74 -> 5.08 mm
- net /D12,MISO: track 32.6 -> 33.6 mm
- net /D11,MOSI: track 30.1 -> 30.8 mm

Commit message: pcb v2 done
Parts:
- D1: value PWR_LED -> PWR
- D2: value D13_LED -> D13
- moved U1 0.30 mm to (-2.50, -12.2)
Routing:
- net GND: track 37.3 -> 36.7 mm
- removed copper zone on F.Cu, net +5V
Other:
- board size 161.8 x 161.8 mm -> 30 x 30 mm
- board text removed: "16MHz"
- board text removed: "Compact ZSS"
- board text removed: "NCP1117"
- board text removed: "atmega328"
- board text removed: "jsh348"

Commit message: update silk screen
Other:
- board text added: "DTR"
- board text added: "GND"
Changed lines of the file:
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@@
   (general
     (thickness 1.6)
-    (drawings 24)
+    (drawings 26)
     (tracks 350)
     (zones 0)
@@
   )
   (setup
-    (last_trace_width 0.3)
+    (last_trace_width 0.13)
     (user_trace_width 0.2)
     (user_trace_width 0.3)
@@
       (effects (font (size 1 1) (thickness 0.15)) (justify mirror))
     )
-    (fp_text value 16MHz (at -0.2 2) (layer B.SilkS)
+    (fp_text value 16MHz (at -0.6 1.9) (layer B.SilkS)
       (effects (font (size 1 1) (thickness 0.15)) (justify mirror))
     )
@@
       (effects (font (size 1 1) (thickness 0.15)))
     )
-    (fp_text value 10K (at 0 1.43 90) (layer F.Fab) hide
+    (fp_text value 10K (at 0.5 -1.4 90) (layer F.SilkS)
       (effects (font (size 1 1) (thickness 0.15)))
     )
@@
     )
   )
+  (gr_text GND (at 12 4) (layer F.SilkS)
+    (effects (font (size 1 1) (thickness 0.15)))
+  )
+  (gr_text DTR (at 12.9 -3.7) (layer F.SilkS)
+    (effects (font (size 1 1) (thickness 0.15)))
+  )
   (gr_circle (center 0 0) (end 15 0) (layer Edge.Cuts) (width 0.15))
